File: eagle/wharehauora-minisensor.brd (EAGLE design)
At the start: 79.1 x 33.4 mm, 21 parts, among them IC1 REG1117

Commit message: Adding in latest version
Parts:
- added JP4: D13 D6 D5, adafruit:1X03
- added R4: 10K, adafruit:R0603
- added SW1: SPST_TACT-EVQQ2, adafruit:EVQ-Q2
- JP2: value (none) -> A0 A1 A2 A3 A4 A5
- moved U1 26.5 mm to (69.9, 29.2), turned to 180 degrees
- moved U$2 0.30 mm to (2.78, 6.35)
Connections:
- new net N$23: R4.1, U$1.33
- new net N$24: JP4.2, U$1.27
- new net N$25: JP4.1, U$1.31
- new net N$26: JP4.3, U$1.32
- net GND: now also R4.2, SW1.A, SW1.A'
- net N$10: now also SW1.B, SW1.B'
Routing:
- net +5V: track 108.3 -> 171.6 mm
- net N$21: track 14.3 -> 46.2 mm
- net N$25: track 0.00 -> 18.5 mm
- net N$24: track 0.00 -> 17.6 mm
- net N$10: track 28.4 -> 39.9 mm
- net N$26: track 0.00 -> 9.47 mm
- net N$6: track 13.2 -> 9.65 mm
- net N$23: track 0.00 -> 2.25 mm
Other:
- board size 79.1 x 33.4 mm -> 79.1 x 33.3 mm
- board text added: "ICSP"
- board text added: "RESET"
- board text added: "Radio"
