File: eagle/wharehauora-minisensor.brd (EAGLE design)
At the start: 79.1 x 33.3 mm, 24 parts, among them IC1 REG1117, SW1 SPST_TACT-EVQQ2

Commit message: Latest board design
Parts:
- added U$3: (no value), creative-commons:CC_TPLACE
- added U$4: (no value), creative-commons:BY_TPLACE
- added U$5: (no value), creative-commons:SA_TPLACE
- Q1: value (none) -> CRYSTALS-NOGND-HC49; device adafruit:HC33U-V -> IQD-Frequency-Products:HC49
- moved C5 7.37 mm to (2.20, 18.3), turned to 180 degrees
- moved C1 6.72 mm to (39.0, 9.08)
- moved C2 4.52 mm to (23.7, 9.08)
- moved Q1 4.35 mm to (31.3, 9.08)
- moved F1 3.10 mm to (9.22, 15.5)
Routing:
- net N$5: track 20.0 -> 10.6 mm
- net N$7: track 16.7 -> 10.6 mm
- net +5V: track 171.6 -> 174.2 mm
Changed lines of the file:
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@@
 <?xml version="1.0" encoding="utf-8"?>
 <!DOCTYPE eagle SYSTEM "eagle.dtd">
-<eagle version="7.7.0">
+<eagle version="7.2.0">
 <drawing>
 <settings>
@@
 <text x="13" y="24.8" size="1.27" layer="125">Radio</text>
 <text x="43.1" y="23.6" size="1.27" layer="125">ICSP</text>
+<hole x="22" y="30" drill="3.2"/>
+<hole x="50.2" y="4" drill="3.2"/>
+<hole x="23.3" y="4" drill="3.2"/>
+<hole x="4.1" y="14" drill="3.2"/>
 </plain>
 <attributes>
@@
 </autorouter>
 <elements>
-<element name="C1" library="eagle-ltspice" package="C0603" value="" x="44.45" y="5.08" smashed="yes" rot="R180">
-<attribute name="SPICEMODEL" value="NONE" x="44.45" y="5.08" size="1.778" layer="27" rot="R180" display="off"/>
-<attribute name="SPICEPREFIX" value="C" x="44.45" y="5.08" size="1.778" layer="27" rot="R180" display="off"/>
-<attribute name="NAME" x="45.585" y="7.545" size="1.27" layer="25" rot="R180"/>
-<attribute name="VALUE" x="45.085" y="6.985" size="1.27" layer="27" rot="R180"/>
-</element>
-<element name="C2" library="eagle-ltspice" package="C0603" value="" x="21.59" y="5.08" smashed="yes">
-<attribute name="SPICEMODEL" value="NONE" x="21.59" y="5.08" size="1.778" layer="27" display="off"/>
-<attribute name="SPICEPREFIX" value="C" x="21.59" y="5.08" size="1.778" layer="27" display="off"/>
-<attribute name="NAME" x="20.455" y="6.315" size="1.27" layer="25"/>
-<attribute name="VALUE" x="20.955" y="3.175" size="1.27" layer="27"/>
+<element name="C1" library="eagle-ltspice" package="C0603" value="" x="39.05" y="9.08" smashed="yes" rot="R180">
+<attribute name="SPICEMODEL" value="NONE" x="39.05" y="9.08" size="1.778" layer="27" rot="R180" display="off"/>
+<attribute name="SPICEPREFIX" value="C" x="39.05" y="9.08" size="1.778" layer="27" rot="R180" display="off"/>
+<attribute name="NAME" x="40.185" y="11.545" size="1.27" layer="25" rot="R180"/>
+<attribute name="VALUE" x="39.685" y="10.985" size="1.27" layer="27" rot="R180"/>
+</element>
+<element name="C2" library="eagle-ltspice" package="C0603" value="" x="23.69" y="9.08" smashed="yes">
+<attribute name="SPICEMODEL" value="NONE" x="23.69" y="9.08" size="1.778" layer="27" display="off"/>
+<attribute name="SPICEPREFIX" value="C" x="23.69" y="9.08" size="1.778" layer="27" display="off"/>
+<attribute name="NAME" x="22.555" y="10.315" size="1.27" layer="25"/>
+<attribute name="VALUE" x="23.055" y="7.175" size="1.27" layer="27"/>
 </element>
 <element name="D1" library="diode" package="SOD80C" value="" x="15.24" y="6.35"/>
 <element name="D2" library="diode" package="SOD80C" value="" x="15.24" y="10.16"/>
-<element name="F1" library="adafruit" package="1812" value="" x="6.12" y="15.54" rot="R90"/>
+<element name="F1" library="adafruit" package="1812" value="" x="9.22" y="15.54" rot="R90"/>
 <element name="IC1" library="burr-brown" package="SOT223" value="REG1117" x="6.22" y="26.76" smashed="yes" rot="R90">
 <attribute name="OC_NEWARK" value="14P6981" x="6.22" y="26.76" size="1.778" layer="27" rot="R90" display="off"/>
@@
 <attribute name="NAME" x="19.545" y="3.17" size="1.27" layer="25" rot="R180"/>
 </element>
-<element name="Q1" library="adafruit" package="HC33U-V" value="" x="33.02" y="5.08">
-<attribute name="OC_NEWARK" value="unknown" x="33.02" y="5.08" size="1.778" layer="27" display="off"/>
-<attribute name="MPN" value="" x="33.02" y="5.08" size="1.778" layer="27" display="off"/>
-<attribute name="MF" value="" x="33.02" y="5.08" size="1.778" layer="27" display="off"/>
-<attribute name="OC_FARNELL" value="unknown" x="33.02" y="5.08" size="1.778" layer="27" display="off"/>
-</element>
+<element name="Q1" library="IQD-Frequency-Products" package="HC49" value="CRYSTALS-NOGND-HC49" x="31.32" y="9.08"/>
 <element name="R1" library="adafruit" package="R0603" value="22R" x="21.59" y="22.86" smashed="yes">
 <attribute name="NAME" x="20.601" y="24.149" size="1.27" layer="25"/>
@@
 <element name="C3" library="rcl" package="C0805" value="" x="3.7" y="21.1" rot="R180"/>
 <element name="C4" library="rcl" package="C0805" value="" x="9.4" y="21.1"/>
-<element name="C5" library="rcl" package="C0603" value="" x="9.5" y="17.3"/>
+<element name="C5" library="rcl" package="C0603" value="" x="2.2" y="18.3" rot="R180"/>
 <element name="C6" library="rcl" package="C0805" value="" x="22.7" y="12.5" rot="R90"/>
 <element name="R4" library="adafruit" package="R0603" value="10K" x="38.4" y="25.3" smashed="yes">
@@
 <attribute name="NAME" x="50.3" y="29.3" size="1.27" layer="25" rot="R270"/>
 </element>
+<element name="U$3" library="creative-commons" package="CC_TPLACE" value="" x="58.7" y="5.9" rot="MR0"/>
+<element name="U$4" library="creative-commons" package="BY_TPLACE" value="" x="47.8" y="5.8" rot="MR0"/>
+<element name="U$5" library="creative-commons" package="SA_TPLACE" value="" x="37" y="5.8" rot="MR0"/>
 </elements>
 <signals>
@@
 <wire x1="5.58" y1="7.65" x2="8.26" y2="7.65" width="0.4064" layer="1"/>
 <wire x1="8.26" y1="7.65" x2="8.26" y2="11.43" width="0.4064" layer="1"/>
-<wire x1="8.26" y1="11.43" x2="7.62" y2="11.43" width="0.4064" layer="1"/>
-<wire x1="7.62" y1="11.43" x2="6.12" y2="13.494" width="0.4064" layer="1"/>
+<wire x1="8.26" y1="11.43" x2="9.22" y2="11.43" width="0.4064" layer="1"/>
+<wire x1="9.22" y1="11.43" x2="9.22" y2="13.494" width="0.4064" layer="1"/>
 </signal>
 <signal name="GND">
@@
 <contactref element="C1" pad="2"/>
 <contactref element="U$1" pad="17"/>
-<wire x1="31.75" y1="13.25" x2="31.75" y2="5.08" width="0.4064" layer="1"/>
-<wire x1="31.75" y1="5.08" x2="39.243" y2="5.08" width="0.4064" layer="1"/>
-<wire x1="39.243" y1="5.08" x2="43.6" y2="5.08" width="0.4064" layer="1"/>
+<wire x1="31.75" y1="13.25" x2="31.75" y2="9.08" width="0.4064" layer="1"/>
+<wire x1="31.75" y1="9.08" x2="33.733" y2="9.08" width="0.4064" layer="1"/>
+<wire x1="33.733" y1="9.08" x2="38.2" y2="9.08" width="0.4064" layer="1"/>
 </signal>
 <signal name="N$7">
@@
 <contactref element="Q1" pad="1"/>
 <contactref element="C2" pad="2"/>
-<wire x1="30.95" y1="13.25" x2="30.95" y2="5.08" width="0.4064" layer="1"/>
-<wire x1="30.95" y1="5.08" x2="26.797" y2="5.08" width="0.4064" layer="1"/>
-<wire x1="26.797" y1="5.08" x2="22.44" y2="5.08" width="0.4064" layer="1"/>
+<wire x1="30.95" y1="13.25" x2="30.95" y2="9.08" width="0.4064" layer="1"/>
+<wire x1="30.95" y1="9.08" x2="28.907" y2="9.08" width="0.4064" layer="1"/>
+<wire x1="28.907" y1="9.08" x2="24.54" y2="9.08" width="0.4064" layer="1"/>
 </signal>
 <signal name="N$10">
@@
 <contactref element="IC1" pad="3"/>
 <contactref element="U1" pad="VDD"/>
-<wire x1="9.3696" y1="29.0714" x2="6.12" y2="29.0714" width="0.4064" layer="1"/>
-<wire x1="6.12" y1="29.0714" x2="6.12" y2="21.1" width="0.4064" layer="1"/>
-<wire x1="6.12" y1="21.1" x2="6.12" y2="17.586" width="0.4064" layer="1"/>
 <wire x1="25.95" y1="22.3" x2="25.95" y2="22.25" width="0.4064" layer="1"/>
 <wire x1="25.95" y1="22.25" x2="27.75" y2="22.25" width="0.4064" layer="1"/>
@@
 <wire x1="50.3" y1="21.1" x2="50.3" y2="21.15" width="0.4064" layer="1"/>
 <contactref element="C3" pad="1"/>
-<wire x1="4.65" y1="21.1" x2="6.12" y2="21.1" width="0.4064" layer="1"/>
-<wire x1="9.3696" y1="29.0714" x2="20.1286" y2="29.0714" width="0.4064" layer="1"/>
-<wire x1="20.1286" y1="29.0714" x2="24.5" y2="24.7" width="0.4064" layer="1"/>
-<wire x1="24.5" y1="24.7" x2="24.5" y2="22.25" width="0.4064" layer="1"/>
+<wire x1="9.3696" y1="29.0714" x2="18.7286" y2="29.0714" width="0.4064" layer="1"/>
+<wire x1="18.7286" y1="29.0714" x2="24.4" y2="23.7" width="0.4064" layer="1"/>
+<wire x1="24.4" y1="23.7" x2="24.5" y2="22.25" width="0.4064" layer="1"/>
 <wire x1="24.5" y1="22.25" x2="25.95" y2="22.25" width="0.4064" layer="1"/>
 <contactref element="C5" pad="1"/>
-<wire x1="6.12" y1="17.586" x2="6.12" y2="17.3" width="0.4064" layer="1"/>
-<wire x1="6.12" y1="17.3" x2="8.65" y2="17.3" width="0.4064" layer="1"/>
 <wire x1="42.51" y1="21.56" x2="42.51" y2="23.3" width="0.4064" layer="1"/>
 <wire x1="42.51" y1="23.3" x2="50.3" y2="23.3" width="0.4064" layer="1"/>
@@
 <wire x1="73.67" y1="15.85" x2="37.55" y2="15.85" width="0.4064" layer="1"/>
 <wire x1="73.67" y1="29.2" x2="73.67" y2="31.1" width="0.4064" layer="1"/>
+<wire x1="9.22" y1="17.586" x2="4.65" y2="17.586" width="0.4064" layer="1"/>
+<wire x1="4.65" y1="17.586" x2="4.65" y2="18.3" width="0.4064" layer="1"/>
+<wire x1="4.65" y1="18.4" x2="4.65" y2="21.1" width="0.4064" layer="1"/>
+<wire x1="4.65" y1="21.1" x2="5.9" y2="21.1" width="0.4064" layer="1"/>
+<wire x1="5.9" y1="21.1" x2="5.9" y2="29" width="0.4064" layer="1"/>
+<wire x1="5.9" y1="29" x2="9.3696" y2="29" width="0.4064" layer="1"/>
+<wire x1="9.3696" y1="29" x2="9.3696" y2="29.0714" width="0.4064" layer="1"/>
+<wire x1="3.05" y1="18.3" x2="4.65" y2="18.3" width="0.4064" layer="1"/>
+<wire x1="4.65" y1="18.3" x2="4.65" y2="18.4" width="0.4064" layer="1"/>
 </signal>
 <signal name="3.3V">
