File: eagle/wharehauora-minisensor.sch (EAGLE design)
At the start: 21 parts, among them IC1 REG1117

Commit message: Adding in latest version
Parts:
- added JP4: D13 D6 D5, adafruit:PINHD-1X3
- added R4: 10K, adafruit:R-US_R0603
- added SW1: SPST_TACT-EVQQ2, adafruit:SPST_TACT-EVQQ2
- JP2: value (none) -> A0 A1 A2 A3 A4 A5
Connections:
- new net N$23: R4.1, U$1.PE2(!HWB)
- new net N$24: JP4.2, U$1.PD7(OC4D/ADC10/T0)
- new net N$25: JP4.1, U$1.PC6(OC3A/!OC4A)
- new net N$26: JP4.3, U$1.PC7(ICP3/CLK0/OC4A)
- net GND: now also R4.2, SW1.P, SW1.P1
- net N$10: now also SW1.S, SW1.S1
Other:
- moved on the sheet: JP2, JP3, R3

Commit message: Latest board design
Parts:
- Q1: value (none) -> CRYSTALS-NOGND-HC49; device adafruit:CRYSTALHC33U-V -> IQD-Frequency-Products:CRYSTALS-NOGND-HC49
Changed lines of the file:
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@@
 <?xml version="1.0" encoding="utf-8"?>
 <!DOCTYPE eagle SYSTEM "eagle.dtd">
-<eagle version="7.7.0">
+<eagle version="7.2.0">
 <drawing>
 <settings>
@@
 <part name="SUPPLY1" library="supply2" deviceset="GND1" device=""/>
 <part name="SUPPLY2" library="supply2" deviceset="GND" device=""/>
-<part name="Q1" library="adafruit" deviceset="CRYSTAL" device="HC33U-V"/>
+<part name="Q1" library="IQD-Frequency-Products" deviceset="CRYSTALS-NOGND" device="-HC49"/>
 <part name="C1" library="eagle-ltspice" deviceset="C" device="C0603"/>
 <part name="C2" library="eagle-ltspice" deviceset="C" device="C0603"/>
